Commit message: Integrated changes made in the master
Integrated changes made in the master on the namespace and other.

File: urdf/wind_turbine.base.urdf.xacro (robot description, xacro)
@@ -18,5 +18,5 @@
         <origin xyz="0 0 0" rpy="0 0 0" />
         <geometry>
-          <mesh filename="package://bebopS/meshes/wind_turbine_base.dae"
+          <mesh filename="package://bebop_simulator/meshes/wind_turbine_base.dae"
             scale="2 2 2" />
         </geometry>
@@ -25,5 +25,5 @@
         <origin xyz="0 0 0" rpy="0 0 0"/>
         <geometry>
-          <mesh filename="package://bebopS/meshes/wind_turbine_base.dae"
+          <mesh filename="package://bebop_simulator/meshes/wind_turbine_base.dae"
             scale="2 2 2" />
         </geometry>
@@ -45,5 +45,5 @@
         <origin xyz="0.16228 -0.00566 0.1" rpy="0 0 0" />
         <geometry>
-          <mesh filename="package://bebopS/meshes/wind_turbine_rotor.dae"
+          <mesh filename="package://bebop_simulator/meshes/wind_turbine_rotor.dae"
             scale="2 2 2" />
         </geometry>
@@ -52,5 +52,5 @@
         <origin xyz="0.16228 -0.00566 0.1" rpy="0 0 0"/>
         <geometry>
-          <mesh filename="package://bebopS/meshes/wind_turbine_rotor.dae"
+          <mesh filename="package://bebop_simultor/meshes/wind_turbine_rotor.dae"
             scale="2 2 2" />
         </geometry>
