Commit message: Removed unnecessary launch files
Removed unnecessary launch file. In addition, the launch files now allow to choose which sensor should be simulated during the flight.

File: urdf/bebop.urdf.xacro (robot description, xacro)
@@ -8,8 +8,14 @@
   <xacro:property name="wind_direction_y" value="$(arg wind_direction_y)" />
   <xacro:property name="wind_direction_z" value="$(arg wind_direction_z)" />
+  <xacro:property name="enable_odometry_sensor_with_noise" value="$(arg enable_odometry_sensor_with_noise)" />
+  <xacro:property name="disable_odometry_sensor_with_noise" value="$(arg disable_odometry_sensor_with_noise)" />
+  <xacro:property name="enable_ground_truth_sensor" value="$(arg enable_ground_truth_sensor)" />
+  <xacro:property name="enable_wind_plugin" value="$(arg enable_wind_plugin)" />
+  <xacro:property name="enable_laser1D" value="$(arg enable_laser1D)" />
   <!-- Instantiate bebop "mechanics" -->
   	<xacro:include filename="$(find bebopS)/urdf/bebop_base.urdf.xacro" />
   	<xacro:include filename="$(find rotors_description)/urdf/component_snippets.xacro" />
-  	<!-- Realistic odometry sensor with noise -->
+  	<!-- Realistic odometry sensor with noise and bias -->
+        <xacro:if value="$(arg enable_odometry_sensor_with_noise)">
 	<xacro:odometry_plugin_macro
 		namespace="${namespace}"
@@ -24,5 +30,37 @@
 		child_frame_id="${namespace}/base_link"
 		mass_odometry_sensor="0.01"
-		measurement_divisor="40"
+		measurement_divisor="4"
+		measurement_delay="0"
+		unknown_delay="0.0"
+		noise_normal_position="0.01 0.01 0.01"
+		noise_normal_quaternion="0.017 0.017 0.017"
+		noise_normal_linear_velocity="0.01 0.01 0.01"
+		noise_normal_angular_velocity="0.01 0.01 0.01"
+		noise_uniform_position="0.0 0.0 0.0"
+		noise_uniform_quaternion="0.0 0.0 0.0"
+		noise_uniform_linear_velocity="0.0 0.0 0.0"
+		noise_uniform_angular_velocity="0.0 0.0 0.0"
+		enable_odometry_map="false"
+		odometry_map=""
+		image_scale="">
+		<inertia ixx="0.00001" ixy="0.0" ixz="0.0" iyy="0.00001" iyz="0.0" izz="0.00001" /> <!-- [kg m^2] [kg m^2] [kg m^2] [kg m^2] [kg m^2] [kg m^2] -->
+		<origin xyz="0.0 0.0 0.0" rpy="0.0 0.0 0.0" />
+	</xacro:odometry_plugin_macro>
+        </xacro:if>
+  	<!-- Realistic odometry sensor without noise and bias -->
+        <xacro:if value="$(arg disable_odometry_sensor_with_noise)">
+	<xacro:odometry_plugin_macro
+		namespace="${namespace}"
+		odometry_sensor_suffix=""
+		parent_link="base_link"
+		pose_topic="pose"
+		pose_with_covariance_topic="pose_with_covariance"
+		position_topic="position"
+		transform_topic="transform"
+		odometry_topic="odometry"
+		parent_frame_id="world"
+		child_frame_id="${namespace}/base_link"
+		mass_odometry_sensor="0.01"
+		measurement_divisor="4"
 		measurement_delay="0"
 		unknown_delay="0.0"
@@ -41,5 +79,7 @@
 		<origin xyz="0.0 0.0 0.0" rpy="0.0 0.0 0.0" />
 	</xacro:odometry_plugin_macro>
-	<!-- Ground truth odometry sensor without noise -->
+        </xacro:if>
+	<!-- Ground truth odometry sensor without noise and bias -->
+        <xacro:if value="$(arg enable_ground_truth_sensor)">
 	<xacro:odometry_plugin_macro
 		namespace="${namespace}"
@@ -71,5 +111,7 @@
 		<origin xyz="0.0 0.0 0.0" rpy="0.0 0.0 0.0" />
 	</xacro:odometry_plugin_macro>
+        </xacro:if>
 	<!-- Instantiate a wind plugin -->
+        <xacro:if value="$(arg enable_wind_plugin)">
 	<gazebo>
 	    <!-- wind plugin -->
@@ -89,51 +131,55 @@
 	    </plugin>
 	</gazebo>
-    <link name="laser1D_link">
-      <inertial>
-        <mass value="1e-5" />
-        <origin xyz="0 0 0" rpy="0 0 0"/>
-        <inertia ixx="1e-6" ixy="0" ixz="0" iyy="1e-6" iyz="0" izz="1e-6" />
-      </inertial>
-    </link>
-    <joint name="laser1D_joint" type="fixed">
-      <!--<axis xyz="0 0 1" />-->
-      <origin xyz="0.111 0 0.0217" rpy="0 0 0"/>
-      <parent link="base_link"/>
-      <child link="laser1D_link"/>
-    </joint>
+        </xacro:if>
+        <!-- Instantiate a laser scanner 1D -->
+        <xacro:if value="$(arg enable_laser1D)">
+	  <link name="laser1D_link">
+	    <inertial>
+	      <mass value="1e-5" />
+	      <origin xyz="0 0 0" rpy="0 0 0"/>
+	      <inertia ixx="1e-6" ixy="0" ixz="0" iyy="1e-6" iyz="0" izz="1e-6" />
+	    </inertial>
+	  </link>
+	  <joint name="laser1D_joint" type="fixed">
+	    <!--<axis xyz="0 0 1" />-->
+	    <origin xyz="0.111 0 0.0217" rpy="0 0 0"/>
+	    <parent link="base_link"/>
+	    <child link="laser1D_link"/>
+	  </joint>
  	<gazebo reference="laser1D_link">
-		<sensor type="ray" name="laser1D_sensor">
-	      <pose>0 0 0 0 0 0</pose>
-	      <visualize>true</visualize>
-	      <update_rate>200</update_rate>
-	      <ray>
-	        <scan>
-	          <horizontal>
-	            <samples>1</samples>
-	            <resolution>1</resolution>
-	            <min_angle>0</min_angle>
-	            <max_angle>0</max_angle>
-	          </horizontal>
-	        </scan>
-	        <range>
-	          <min>0.10</min>
-	          <max>100.0</max>
-	          <resolution>0.01</resolution>
-	        </range>
-	        <noise>
-	          <type>gaussian</type>
-	          <!-- Noise parameters based on published spec for Hokuyo laser
+	  <sensor type="ray" name="laser1D_sensor">
+	    <pose>0 0 0 0 0 0</pose>
+	    <visualize>true</visualize>
+	    <update_rate>200</update_rate>
+	    <ray>
+	      <scan>
+	        <horizontal>
+	          <samples>1</samples>
+	          <resolution>1</resolution>
+	          <min_angle>0</min_angle>
+	          <max_angle>0</max_angle>
+	        </horizontal>
+	      </scan>
+	      <range>
+	        <min>0.10</min>
+	        <max>100.0</max>
+	        <resolution>0.01</resolution>
+	      </range>
+	      <noise>
+	       <type>gaussian</type>
+	         <!-- Noise parameters based on published spec for Hokuyo laser
 	               achieving "+-30mm" accuracy at range < 10m.  A mean of 0.0m and
 	               stddev of 0.01m will put 99.7% of samples within 0.03m of the true
 	               reading. -->
-	          <mean>0.0</mean>
-	          <stddev>0.01</stddev>
-	        </noise>
-	      </ray>
-	      <plugin name="gazebo_ros_head_hokuyo_controller" filename="libgazebo_ros_laser.so">
-	        <topicName>laser/scan</topicName>
-	        <frameName>laser1D_link</frameName>
-	      </plugin>
-	    </sensor>
+	        <mean>0.0</mean>
+	        <stddev>0.01</stddev>
+	      </noise>
+	    </ray>
+	    <plugin name="gazebo_ros_head_hokuyo_controller" filename="libgazebo_ros_laser.so">
+	     <topicName>laser/scan</topicName>
+	     <frameName>laser1D_link</frameName>
+	    </plugin>
+	   </sensor>
   	</gazebo>
-</robot>
+     </xacro:if>
+ </robot>

Commit message: Fixed namespace

File: urdf/bebop.urdf.xacro (robot description, xacro)
@@ -14,5 +14,5 @@
   <xacro:property name="enable_laser1D" value="$(arg enable_laser1D)" />
   <!-- Instantiate bebop "mechanics" -->
-  	<xacro:include filename="$(find bebopS)/urdf/bebop_base.urdf.xacro" />
+  	<xacro:include filename="$(find bebop_simulator)/urdf/bebop_base.urdf.xacro" />
   	<xacro:include filename="$(find rotors_description)/urdf/component_snippets.xacro" />
   	<!-- Realistic odometry sensor with noise and bias -->

File: urdf/bebop_base.urdf.xacro (robot description, xacro)
@@ -34,5 +34,5 @@
   </xacro:property>
   <!-- Included URDF Files -->
-  <xacro:include filename="$(find bebopS)/urdf/multirotor_base.urdf.xacro" />
+  <xacro:include filename="$(find bebop_simulator)/urdf/multirotor_base.urdf.xacro" />
   <!-- Instantiate multirotor_base_macro once -->
   <xacro:multirotor_base_macro

File: urdf/multirotor_base.urdf.xacro (robot description, xacro)
@@ -19,5 +19,5 @@
         <origin xyz="0 0 0" rpy="0 0 0" />
         <geometry>
-          <mesh filename="package://bebopS/meshes/${mesh_file}"
+          <mesh filename="package://bebop_simulator/meshes/${mesh_file}"
             scale="0.001 0.001 0.001" />
           <!-- <box size="${body_width} ${body_width} ${body_height}"/> --> <!-- [m] [m] [m] -->
@@ -78,5 +78,5 @@
         <geometry>
           <!-- <cylinder length="0.005" radius="${radius_rotor}"/> --> <!-- [m] -->
-          <mesh filename="package://bebopS/meshes/propeller_${direction}.dae"
+          <mesh filename="package://bebop_simulator/meshes/propeller_${direction}.dae"
             scale="0.00055 0.00055 0.00055" />
           <!-- <box size="${2*radius_rotor} 0.01 0.005"/> -->

File: urdf/wind_turbine.base.urdf.xacro (robot description, xacro)
@@ -18,5 +18,5 @@
         <origin xyz="0 0 0" rpy="0 0 0" />
         <geometry>
-          <mesh filename="package://bebopS/meshes/wind_turbine_base.dae"
+          <mesh filename="package://bebop_simulator/meshes/wind_turbine_base.dae"
             scale="2 2 2" />
         </geometry>
@@ -25,5 +25,5 @@
         <origin xyz="0 0 0" rpy="0 0 0"/>
         <geometry>
-          <mesh filename="package://bebopS/meshes/wind_turbine_base.dae"
+          <mesh filename="package://bebop_simulator/meshes/wind_turbine_base.dae"
             scale="2 2 2" />
         </geometry>
@@ -45,5 +45,5 @@
         <origin xyz="0.16228 -0.00566 0.1" rpy="0 0 0" />
         <geometry>
-          <mesh filename="package://bebopS/meshes/wind_turbine_rotor.dae"
+          <mesh filename="package://bebop_simulator/meshes/wind_turbine_rotor.dae"
             scale="2 2 2" />
         </geometry>
@@ -52,5 +52,5 @@
         <origin xyz="0.16228 -0.00566 0.1" rpy="0 0 0"/>
         <geometry>
-          <mesh filename="package://bebopS/meshes/wind_turbine_rotor.dae"
+          <mesh filename="package://bebop_simulator/meshes/wind_turbine_rotor.dae"
             scale="2 2 2" />
         </geometry>

File: urdf/wind_turbine.gazebo.xacro (robot description, xacro)
@@ -15,5 +15,5 @@
   <xacro:property name="bag_file" value="wind_turbine.bag" />
   <!-- Instantiate mmuav "mechanics" -->
-  <xacro:include filename="$(find bebopS)/urdf/wind_turbine.base.urdf.xacro" />
+  <xacro:include filename="$(find bebop_simulator)/urdf/wind_turbine.base.urdf.xacro" />
   <xacro:include filename="$(find rotors_description)/urdf/component_snippets.xacro" />
 </robot>

Commit message: Add default IMU sensor

File: urdf/bebop.urdf.xacro (robot description, xacro)
@@ -9,4 +9,5 @@
   <xacro:property name="wind_direction_z" value="$(arg wind_direction_z)" />
   <xacro:property name="enable_odometry_sensor_with_noise" value="$(arg enable_odometry_sensor_with_noise)" />
+  <xacro:property name="enable_imu" value="$(arg enable_imu)" />
   <xacro:property name="disable_odometry_sensor_with_noise" value="$(arg disable_odometry_sensor_with_noise)" />
   <xacro:property name="enable_ground_truth_sensor" value="$(arg enable_ground_truth_sensor)" />
@@ -47,4 +48,27 @@
 		<origin xyz="0.0 0.0 0.0" rpy="0.0 0.0 0.0" />
 	</xacro:odometry_plugin_macro>
+        </xacro:if>
+        <!-- RotorS default IMU -->
+        <xacro:if value="$(arg enable_imu)">
+	<!-- ADIS16448 IMU. -->
+	<xacro:imu_plugin_macro
+		namespace="${namespace}"
+		imu_suffix=""
+		parent_link="base_link"
+		imu_topic="imu"
+		measurement_delay="0"
+		measurement_divisor="1"
+		mass_imu_sensor="0.015"
+		gyroscope_noise_density="0.0003394"
+		gyroscope_random_walk="0.000038785"
+		gyroscope_bias_correlation_time="1000.0"
+		gyroscope_turn_on_bias_sigma="0.0087"
+		accelerometer_noise_density="0.004"
+		accelerometer_random_walk="0.006"
+		accelerometer_bias_correlation_time="300.0"
+		accelerometer_turn_on_bias_sigma="0.1960">
+		<inertia ixx="0.00001" ixy="0.0" ixz="0.0" iyy="0.00001" iyz="0.0" izz="0.00001" />
+		<origin xyz="0 0 0" rpy="0 0 0" />
+	</xacro:imu_plugin_macro>
         </xacro:if>
   	<!-- Realistic odometry sensor without noise and bias -->

Commit message: Insert IMU in the available sensors for the Bebop
Inserted the IMU in the list of the available sensors of the vehicle

File: urdf/bebop.urdf.xacro (robot description, xacro)
@@ -47,4 +47,27 @@
 		<origin xyz="0.0 0.0 0.0" rpy="0.0 0.0 0.0" />
 	</xacro:odometry_plugin_macro>
+        </xacro:if>
+        <!-- RotorS default IMU -->
+        <xacro:if value="$(arg enable_imu)">
+	<!-- ADIS16448 IMU. -->
+	<xacro:imu_plugin_macro
+		namespace="${namespace}"
+		imu_suffix=""
+		parent_link="base_link"
+		imu_topic="imu"
+		measurement_delay="0"
+		measurement_divisor="1"
+		mass_imu_sensor="0.015"
+		gyroscope_noise_density="0.0003394"
+		gyroscope_random_walk="0.000038785"
+		gyroscope_bias_correlation_time="1000.0"
+		gyroscope_turn_on_bias_sigma="0.0087"
+		accelerometer_noise_density="0.004"
+		accelerometer_random_walk="0.006"
+		accelerometer_bias_correlation_time="300.0"
+		accelerometer_turn_on_bias_sigma="0.1960">
+		<inertia ixx="0.00001" ixy="0.0" ixz="0.0" iyy="0.00001" iyz="0.0" izz="0.00001" />
+		<origin xyz="0 0 0" rpy="0 0 0" />
+	</xacro:imu_plugin_macro>
         </xacro:if>
   	<!-- Realistic odometry sensor without noise and bias -->
