Commit message: Spaces

File: urdf/multirotor_base.urdf.xacro (robot description, xacro)
@@ -85,4 +85,5 @@
       <collision>
         <geometry>
+          <!-- <cylinder length="0.005" radius="${radius_rotor}"/> --> <!-- [m] -->
           <cylinder length="0.005" radius="${radius_rotor}" /> <!-- [m] -->
         </geometry>

Commit message: Changes propagation #29

File: urdf/multirotor_base.urdf.xacro (robot description, xacro)
@@ -85,5 +85,4 @@
       <collision>
         <geometry>
-          <!-- <cylinder length="0.005" radius="${radius_rotor}"/> --> <!-- [m] -->
           <cylinder length="0.005" radius="${radius_rotor}" /> <!-- [m] -->
         </geometry>
@@ -100,9 +99,9 @@
         <motorConstant>${motor_constant}</motorConstant>
         <momentConstant>${moment_constant}</momentConstant>
-        <commandTopic>${robot_namespace}/command/motors</commandTopic>
+        <commandSubTopic>${robot_namespace}/command/motors</commandSubTopic>
         <motorNumber>${motor_number}</motorNumber>
         <rotorDragCoefficient>${rotor_drag_coefficient}</rotorDragCoefficient>
         <rollingMomentCoefficient>${rolling_moment_coefficient}</rollingMomentCoefficient>
-        <motorVelocityTopic>${robot_namespace}/motor_vel/${motor_number}</motorVelocityTopic>
+        <motorSpeedPubTopic>${robot_namespace}/motor_vel/${motor_number}</motorSpeedPubTopic>
         <rotorVelocitySlowdownSim>${rotor_velocity_slowdown_sim}</rotorVelocitySlowdownSim>
       </plugin>
